File: Electronics/components/resistors/series-parallel/resistors_series_parallel_Rb1.kicad_sch (KiCad schematic)
At the start: 8 parts

Commit message: new schematics visualyse coculation progress resisitors series parallel folder
Parts:
- removed R4: 300, symbol Device:R
- Rb1: value 1k -> 230.769
Changed lines of the file:
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@@
-	)
-	(junction
-		(at 85.09 25.4)
-		(diameter 0)
-		(color 0 0 0 0)
 	)
 	(junction
@@
 	)
 	(junction
-		(at 101.6 38.1)
-		(diameter 0)
-		(color 0 0 0 0)
-	)
-	(junction
 		(at 68.58 46.99)
-		(diameter 0)
-		(color 0 0 0 0)
-	)
-	(junction
-		(at 92.71 25.4)
-		(diameter 0)
-		(color 0 0 0 0)
-	)
-	(junction
-		(at 76.2 38.1)
 		(diameter 0)
 		(color 0 0 0 0)
@@
 	(wire
 		(pts
-			(xy 92.71 38.1) (xy 101.6 38.1)
+			(xy 92.71 38.1) (xy 109.22 38.1)
 		)
 		(stroke
@@
 	(wire
 		(pts
-			(xy 101.6 38.1) (xy 109.22 38.1)
-		)
-		(stroke
-			(width 0)
-			(type default)
-		)
-	)
-	(wire
-		(pts
 			(xy 52.07 38.1) (xy 68.58 38.1)
 		)
@@
 	(wire
 		(pts
-			(xy 68.58 38.1) (xy 76.2 38.1)
+			(xy 68.58 38.1) (xy 85.09 38.1)
 		)
 		(stroke
@@
 	(wire
 		(pts
-			(xy 85.09 25.4) (xy 76.2 25.4)
-		)
-		(stroke
-			(width 0)
-			(type default)
-		)
-	)
-	(wire
-		(pts
-			(xy 101.6 25.4) (xy 101.6 38.1)
-		)
-		(stroke
-			(width 0)
-			(type default)
-		)
-	)
-	(wire
-		(pts
 			(xy 121.92 38.1) (xy 121.92 59.69)
 		)
@@
 	(wire
 		(pts
-			(xy 76.2 25.4) (xy 76.2 38.1)
-		)
-		(stroke
-			(width 0)
-			(type default)
-		)
-	)
-	(wire
-		(pts
-			(xy 86.36 25.4) (xy 85.09 25.4)
-		)
-		(stroke
-			(width 0)
-			(type default)
-		)
-	)
-	(wire
-		(pts
 			(xy 85.09 38.1) (xy 86.36 38.1)
 		)
@@
 	(wire
 		(pts
-			(xy 92.71 25.4) (xy 101.6 25.4)
-		)
-		(stroke
-			(width 0)
-			(type default)
-		)
-	)
-	(wire
-		(pts
-			(xy 76.2 38.1) (xy 85.09 38.1)
-		)
-		(stroke
-			(width 0)
-			(type default)
-		)
-	)
-	(wire
-		(pts
 			(xy 121.92 59.69) (xy 121.92 60.96)
 		)
@@
 		(pts
 			(xy 50.8 38.1) (xy 52.07 38.1)
-		)
-		(stroke
-			(width 0)
-			(type default)
-		)
-	)
-	(wire
-		(pts
-			(xy 91.44 25.4) (xy 92.71 25.4)
 		)
 		(stroke
@@
 		)
 		(instances
-			(project "resistors_series_parallel_combined"
+			(project "resistors_series_parallel_Rb1 - Copy"
 				(path "/ae436056-4544-44d2-91a0-fceb0c77bc0a"
 					(reference "BT1")
@@
 		)
 		(instances
-			(project "resistors_series_parallel_combined"
+			(project "resistors_series_parallel_Rb1 - Copy"
 				(path "/ae436056-4544-44d2-91a0-fceb0c77bc0a"
 					(reference "R1")
@@
 			)
 		)
-		(property "Value" "1k"
+		(property "Value" "230.769"
 			(at 88.9 34.29 90)
 			(show_name no)
@@
 		)
 		(instances
-			(project "resistors_series_parallel_combined"
+			(project "resistors_series_parallel_Rb1 - Copy"
 				(path "/ae436056-4544-44d2-91a0-fceb0c77bc0a"
 					(reference "Rb1")
@@
 		)
 		(instances
-			(project "resistors_series_parallel_combined"
+			(project "resistors_series_parallel_Rb1 - Copy"
 				(path "/ae436056-4544-44d2-91a0-fceb0c77bc0a"
 					(reference "R7")
-					(unit 1)
-				)
-			)
-		)
-	)
-	(symbol
-		(lib_id "Device:R")
-		(at 88.9 25.4 270)
-		(unit 1)
-		(body_style 1)
-		(exclude_from_sim no)
-		(in_bom yes)
-		(on_board yes)
-		(in_pos_files yes)
-		(dnp no)
-		(fields_autoplaced yes)
-		(property "Reference" "R4"
-			(at 88.9 19.05 90)
-			(show_name no)
-			(do_not_autoplace no)
-			(effects
-				(font
-					(size 1.27 1.27)
-				)
-			)
-		)
-		(property "Value" "300"
-			(at 88.9 21.59 90)
-			(show_name no)
-			(do_not_autoplace no)
-			(effects
-				(font
-					(size 1.27 1.27)
-				)
-			)
-		)
-		(property "Footprint" ""
-			(at 88.9 23.622 90)
-			(hide yes)
-			(show_name no)
-			(do_not_autoplace no)
-			(effects
-				(font
-					(size 1.27 1.27)
-				)
-			)
-		)
-		(property "Datasheet" ""
-			(at 88.9 25.4 0)
-			(hide yes)
-			(show_name no)
-			(do_not_autoplace no)
-			(effects
-				(font
-					(size 1.27 1.27)
-				)
-			)
-		)
-		(property "Description" "Resistor"
-			(at 88.9 25.4 0)
-			(hide yes)
-			(show_name no)
-			(do_not_autoplace no)
-			(effects
-				(font
-					(size 1.27 1.27)
-				)
-			)
-		)
-		(pin "2"
-		)
-		(pin "1"
-		)
-		(instances
-			(project "resistors_series_parallel_combined"
-				(path "/ae436056-4544-44d2-91a0-fceb0c77bc0a"
-					(reference "R4")
 					(unit 1)
 				)
@@
 		)
 		(instances
-			(project "resistors_series_parallel_combined"
+			(project "resistors_series_parallel_Rb1 - Copy"
 				(path "/ae436056-4544-44d2-91a0-fceb0c77bc0a"
 					(reference "R2")
@@
 		)
 		(instances
-			(project "resistors_series_parallel_combined"
+			(project "resistors_series_parallel_Rb1 - Copy"
 				(path "/ae436056-4544-44d2-91a0-fceb0c77bc0a"
 					(reference "R6")
@@
 		)
 		(instances
-			(project "resistors_series_parallel_combined"
+			(project "resistors_series_parallel_Rb1 - Copy"
 				(path "/ae436056-4544-44d2-91a0-fceb0c77bc0a"
 					(reference "R3")
