File: Electronics/components/resistors/series-parallel/resistors_series_parallel_Rb2.kicad_sch (KiCad schematic)
At the start: 8 parts

Commit message: new schematics visualyse coculation progress resisitors series parallel folder
Parts:
- removed R4: 300, symbol Device:R
- removed R7: 500, symbol Device:R
- Rb1: value 1k -> 230.769
- Rb2: renamed from R6; value 2K -> 400
